File: Will PCB/ledstatus.kicad_pcb (KiCad board)
At the start: 2 copper layers, 10.2 x 46.7 mm, 11 parts, among them IC1 ATTINY25-P, P1 CONN_1, P2 CONN_1, SW1 SW_PUSH, SW2 SW_PUSH

Commit message: New PCBs
Parts:
- turned R3 to 180 degrees
Routing:
- net N-000006: track 8.69 -> 24.5 mm, vias 0 -> 2
- net N-000009: track 27.1 -> 12.9 mm, vias 1 -> 0
- net N-000005: track 7.35 -> 18.4 mm, vias 0 -> 1
- net GND: track 64.6 -> 66.8 mm
- net N-0000010: track 12.4 -> 14.3 mm
- net N-000004: track 32.6 -> 33.9 mm, vias 3 -> 1
- net N-000001: track 4.02 -> 3.26 mm
- net N-000008: track 13.5 -> 13.7 mm, vias 2 -> 1
Other:
- board text added: "Pato & Will LEDStatusIndicator v1.3"
